Commit message: start branch :: merged torque control by Mr.Kojima and estimate virtual force by Mr.Hiraoka

File: hrpsys_ros_bridge_tutorials/models/JAXON_RED.urdf.xacro (robot description, xacro)
@@ -60,5 +60,6 @@
     <!-- <origin xyz="0.097542410 -0.000296955 0.063307448" rpy="-0.007600616 0.046755703 -0.015569626" /> -->
     <!-- 2016.6.1 tamura kumagai by modification of mount frame -->
-    <origin rpy="-0.005 0.048 -0.020569626" xyz="0.095 0.003596955 0.075307448"/>
+    <!-- <origin rpy="-0.005 0.048 -0.020569626" xyz="0.095 0.003596955 0.075307448"/> -->
+    <origin rpy="-0.004 0.275 -0.01" xyz="0.1 0.01 0.085"/>
   </joint>
   <!-- for calibration / original offset of camera_frame
